Commit message: changes for appras_bearcar_2024

File: realsense2_description/urdf/_r430.urdf.xacro (robot description, xacro)
@@ -1,19 +1,6 @@
 <?xml version="1.0"?>
 <!--
-# Copyright 2023 Intel Corporation. All Rights Reserved.
-#
-# Licensed under the Apache License, Version 2.0 (the "License");
-# you may not use this file except in compliance with the License.
-# You may obtain a copy of the License at
-#
-#     http://www.apache.org/licenses/LICENSE-2.0
-#
-# Unless required by applicable law or agreed to in writing, software
-# distributed under the License is distributed on an "AS IS" BASIS,
-# WITHOUT WARRANTIES OR CONDITIONS OF ANY KIND, either express or implied.
-# See the License for the specific language governing permissions and
-# limitations under the License.
--->
-<!--
+License: Apache 2.0. See LICENSE file in root directory.
+Copyright(c) 2022 Intel Corporation. All Rights Reserved
 This is the URDF model for the Intel RealSense 430 camera, in it's
 aluminum peripherial evaluation case.
@@ -28,4 +15,5 @@
   <xacro:property name="r430_cam_depth_to_infra1_offset" value="-0.025"/>
   <xacro:property name="r430_cam_depth_to_infra2_offset" value="0.025"/>
+  <xacro:property name="r430_cam_depth_to_fisheye_offset" value="0.042"/>
   <!-- The following values model the aluminum peripherial case for the
     R430 camera, with the camera joint represented by the actual
@@ -51,5 +39,5 @@
         <geometry>
           <box size="${r430_cam_width} ${r430_cam_height} ${r430_cam_depth}"/>
-          <!--<mesh filename="file://$(find realsense2_description)/meshes/r430/r430.dae" />-->
+          <!--<mesh filename="package://realsense2_description/meshes/r430/r430.dae" />-->
         </geometry>
         <material name="aluminum"/>
@@ -109,4 +97,17 @@
       </joint>
       <link name="${name}_infra2_optical_frame"/>
+      <!-- camera fisheye joints and links -->
+      <joint name="${name}_fisheye_joint" type="fixed">
+        <origin xyz="0 ${r430_cam_depth_to_fisheye_offset} 0" rpy="0 0 0" />
+        <parent link="${name}_depth_frame" />
+        <child link="${name}_fisheye_frame" />
+      </joint>
+      <link name="${name}_fisheye_frame"/>
+      <joint name="${name}_fisheye_optical_joint" type="fixed">
+        <origin xyz="0 0 0" rpy="${-M_PI/2} 0 ${-M_PI/2}" />
+        <parent link="${name}_fisheye_frame" />
+        <child link="${name}_fisheye_optical_frame" />
+      </joint>
+      <link name="${name}_fisheye_optical_frame"/>
     </xacro:if>
   </xacro:macro>
